File: PCM5242-Julian 2.10/PCM5242/PCM5242.kicad_sch (KiCad schematic)
At the start: 37 parts, among them IC1 NCP163ASN330T1G, IC2 NCP163ASN330T1G, J1 Conn_01x10_Male, J2 Conn_01x10_Male, J3 Conn_01x03_Male, U1 PCM5242, Y1 ASE-24.000MHZ-ET

Commit message: Add files via upload
Some progress was made on the PCB and schematic should be finished. Everything is placed, now I need to route and make the ground pours.
Parts:
- removed C3: 0.1uF, Capacitor_SMD:C_0603_1608Metric_Pad1.08x0.95mm_HandSolder, symbol Device:C
- removed J1, J2: Conn_01x10_Male, Connector_PinHeader_2.54mm:PinHeader_1x10_P2.54mm_Vertical, symbol Connector:Conn_01x10_Male
- removed R1: 10k, Resistor_SMD:R_1206_3216Metric_Pad1.30x1.75mm_HandSolder, symbol Device:R
- added J1: Conn_01x04_Male, Connector_PinHeader_2.54mm:PinHeader_1x04_P2.54mm_Vertical, symbol Connector:Conn_01x04_Male
- added J2: Conn_01x12_Male, Connector_PinHeader_2.54mm:PinHeader_1x12_P2.54mm_Vertical, symbol Connector:Conn_01x12_Male
- C4: value 2.2uF -> 0.1uF
Connections:
- net A16 is gone; now on net A14: U1.31 (LRCK)
- net A17 is gone; now on net A15: U1.32 (ADR1)
- net XSMT is gone; now on net AVDD: U1.1 (XSMT)
- net A10: now also J2.7 (Pin_7)
- net A11: now also U1.25 (GPIO6), J2.8 (Pin_8); no longer U1.23 (MODE1)
- net A12: now also U1.27 (BCK), J2.9 (Pin_9); no longer U1.24 (MODE2)
- net A13: now also U1.28 (DIN), J2.10 (Pin_10); no longer U1.25 (GPIO6)
- net A14: now also J2.11 (Pin_11); no longer U1.27 (BCK)
- net A15: now also J2.12 (Pin_12); no longer U1.28 (DIN)
- net A2: now also J1.2 (Pin_2)
- net A3: now also J1.3 (Pin_3)
- net A4: now also R11.1, J1.4 (Pin_4); no longer R11.2, R7.2
- net A5: now also J2.2 (Pin_2)
- net A6: now also J2.3 (Pin_3)
- net A7: now also J2.4 (Pin_4)
- net A8: now also J2.5 (Pin_5)
- net A9: now also J2.6 (Pin_6)
- net AVDD: now also C1.1, C4.1, U1.5 (CPVDD)
- net DVDD: now also U1.24 (MODE2)
- net GNDD: now also U1.23 (MODE1), J2.1 (Pin_1); no longer R10.1, R11.1
- net VCC: no longer C1.1, C4.1, U1.5 (CPVDD)
- net No Connect: now reaches U1.29 (NC)
- net No Connect: now also U1.30 (NC)
- new net: R11.2, R7.2
- new net A1: J1.1 (Pin_1), R10.1
Other:
- note added: "Analog Out"
- note added: "Digital Out"
- note added: "Power In / Analog Ground"
- note removed: "Digital"
- moved on the sheet: J3, R11, R6
