File: IOBoard/IO Board.kicad_sch (KiCad schematic)
At the start: 25 parts, among them U1 AP2112K-3.3, U2 ATSAMD09D14A-M

Commit message: IOBoard PCB v1
Parts:
- removed J?: Conn_01x06_Male, symbol Connector:Conn_01x06_Male
- removed SW? (x4): SW_DIP_x01, symbol Switch:SW_DIP_x01
- added C4: 10u, Capacitor_SMD:C_0201_0603Metric, symbol Device:C_Small
- added C5: 0.1u, Capacitor_SMD:C_0201_0603Metric, symbol Device:C_Small
- added J1, J2: Conn_01x04_Male, Connector_PinHeader_2.54mm:PinHeader_1x04_P2.54mm_Vertical, symbol Connector:Conn_01x04_Male
- added S1, S2, S3, S4: EG1218, digikey-footprints:Switch_Slide_11.6x4mm_EG1218, symbol dk_Slide-Switches:EG1218
- C1, C2, C3: footprint (none) -> Capacitor_SMD:C_0201_0603Metric
- D1, D2, D3, D4: renamed from D?; footprint (none) -> LED_THT:LED_D3.0mm
- ENC0, ENC1, ENC2, ENC3: footprint (none) -> Rotary_Encoder:RotaryEncoder_Bourns_Vertical_PEC12R-3xxxF-Sxxxx
- R1: footprint (none) -> Resistor_SMD:R_0603_1608Metric
- R2, R3, R4, R5, R6: renamed from R?; footprint (none) -> Resistor_SMD:R_0603_1608Metric
- gave numbers to parts that had none: 1
Connections:
- net +3.3V: now also C2.2, C3.2, C4.2, C5.2, S1.2, S2.2, S3.2, S4.2; no longer C2.1, C3.1
- net ENC0_A: now also U2.2 (PA03); no longer U2.1 (PA02)
- net ENC0_B: now also U2.1 (PA02); no longer U2.2 (PA03)
- net ENC0_SW: now also U2.3 (PA04); no longer U2.11 (PA14)
- net ENC1_A: now also U2.8 (PA09/XOUT); no longer U2.3 (PA04)
- net ENC1_B: now also ENC1.B, U2.7 (PA08/XIN); no longer U2.4 (PA05)
- net ENC1_SW: now also U2.9 (PA10); no longer U2.12 (PA15)
- net ENC2_A: now also U2.16 (PA23); no longer U2.15 (PA22)
- net ENC2_B: now also U2.15 (PA22); no longer U2.16 (PA23)
- net ENC2_SW: now also U2.14 (PA17); no longer U2.13 (PA16)
- net ENC3_A: now also U2.12 (PA15); no longer U2.9 (PA10)
- net ENC3_B: now also U2.11 (PA14); no longer U2.10 (PA11)
- net ENC3_SW: now also U2.10 (PA11); no longer U2.14 (PA17)
- net GND: now also C2.1, C3.1, C4.1, C5.1, J2.2 (Pin_2); no longer C2.2, C3.2
- net SCL: now also J2.4 (Pin_4)
- net SDA: now also J2.3 (Pin_3)
- net SW0: now also S1.1
- net SW1: now also S2.1
- net SW2: now also S3.1
- net SW3: now also S4.1
- net SWCLK0: now also J1.2 (Pin_2)
- net SWCLK1: now also J1.3 (Pin_3)
- net SWDIO0: now also J1.1 (Pin_1)
- net SWDIO1: now also J1.4 (Pin_4)
- net VCC: now also J2.1 (Pin_1)
Other:
- note added: "I2C Headers"
- note added: "Programming Header"
- note removed: "Header"
- moved on the sheet: R1, R5, U2, U3
