File: IOBoard_ATSAMD21/IOBoard_ATSAMD21.kicad_sch (KiCad schematic)
At the start: 36 parts, among them J1 Conn_PIC_ICSP_ICD, J2 Conn_01x04_Male, SW1 EG_1218, SW2 EG_1218, SW3 EG_1218, SW4 EG_1218, U1 ATSAMD21G18A-A, U2 AP2112K-3.3

Commit message: IO Board Silkscreening Finished
Parts:
- removed R6, R7, R8, R9: 10k, Resistor_SMD:R_0603_1608Metric, symbol Device:R_Small
- added H1: MountingHole_Pad, symbol Mechanical:MountingHole_Pad
- added H2, H3, H4: MountingHole_Pad, MountingHole:MountingHole_2.2mm_M2_Pad, symbol Mechanical:MountingHole_Pad
Connections:
- net GND: now also H1.1, H2.1, H3.1, H4.1
- net SW0: now also SW1.2
- net SW1: now also SW2.2
- net SW2: now also SW3.2
- net SW3: now also SW4.2
Other:
- note added: "Bypass Capacitors"
- note added: "Mounting Holes"
