File: IOBoard_ATSAMD21/IOBoard_ATSAMD21.kicad_sch (KiCad schematic)
At the start: 70 parts, among them J1 Conn_PIC_ICSP_ICD, J13 Eurorack_Mono_Jack, J5 Conn_01x05_Pin, J6 Conn_02x03_Odd_Even, SW1 EG_1218, SW2 EG_1218, SW3 EG_1218, SW4 EG_1218, U1 ATSAMD21G18A-A, U2 AP2112K-3.3, U3 ${SIM.PARAMS}, U6 ${SIM.PARAMS}, U7 ${SIM.PARAMS}

Commit message: giving up on differential for now
Parts:
- removed J5: Conn_01x05_Pin, symbol Connector:Conn_01x05_Pin
- removed U3, U6, U7: ${SIM.PARAMS}, Package_SO:SOIC-8_3.9x4.9mm_P1.27mm, symbol Simulation_SPICE:OPAMP
- added FB1: FerriteBead, Inductor_SMD:L_0603_1608Metric_Pad1.05x0.95mm_HandSolder, symbol Device:FerriteBead
- added J5, J9: Conn_01x03_Pin, Connector_PinHeader_2.54mm:PinHeader_1x03_P2.54mm_Vertical, symbol Connector:Conn_01x03_Pin
- added U3, U9: LM2904, Package_SO:SOIC-8_3.9x4.9mm_P1.27mm, symbol Amplifier_Operational:LM2904
- J6: footprint (none) -> Connector_PinHeader_2.54mm:PinHeader_2x03_P2.54mm_Vertical
Connections:
- net +3.3V: now also U9.8 (V+)
- net ADC_in: now also J9.3 (Pin_3)
- net Audio_out: now also U3.1
- net CV_out: now also U9.7
- net GND: no longer C1.1, C10.2, C11.1, C2.1, C3.2, C4.1, C5.2, C6.2, C7.1, C8.2, C9.1, ENC0.C, ENC1.C, ENC2.C, ENC3.C, H1.1, H2.1, H3.1, H4.1, J1.3 (VSS), R1.1, R2.1, R3.1, R4.1, U2.2 (GND)
- net GNDA: now also C1.1, C2.1, ENC0.C, ENC1.C, ENC2.C, ENC3.C, H3.1, H4.1, FB1.2, J5.2 (Pin_2)
- net LL_out: now also U9.1
- net SCL: now also J9.1 (Pin_1)
- net SDA: now also J9.2 (Pin_2)
- net VCC: now also J5.1 (Pin_1), U3.8 (V+)
- net at C16.2, C17.2, C18.2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: now also U9.6 (-)
- net at R12.1: now also U9.5 (+)
- net at C13.2, C14.2, R10.2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: now also U9.2 (-)
- net at R17.1: now also U3.3 (+)
- net at C21.2, R15.2, R18.2: now also U3.2 (-)
- net at R9.1: now also U9.3 (+)
- new net GNDD: C10.2, C11.1, C3.2, C4.1, C5.2, C6.2, C7.1, C8.2, C9.1, FB1.1, H1.1, H2.1, J1.3 (VSS), J5.3 (Pin_3), R1.1, R2.1, R3.1, R4.1, U2.2 (GND), U3.4 (V-), U9.4 (V-)
- no-connect marks 3 -> 22
Other:
- note added: "Amp Jumpers"
- note added: "Amp Power"
- note added: "Can change which holes are GNDA and GNDD"
- note added: "DAC Output Amp"
- note added: "DAC amp"
- note added: "Ferrite Bead"
- note added: "Input amp"
- note added: "Other half of op-amp chip"
- note removed: "Amp jumpers"
- note removed: "Output Amp"
- moved on the sheet: S3

Commit message: IOBoard v3 WIP
Parts:
- ENC0, ENC1, ENC2, ENC3: footprint custom_lib:PEC12R-3217F-S0024-ND -> customlib:PEC12R-3217F-S0024-ND
- S1, S2, S3: footprint digikey-footprints:Switch_Slide_11.6x4mm_EG1218 -> customlib:EG_1218
- SW1, SW2, SW3, SW4: footprint custom_lib:EG_1218 -> customlib:EG_1218
Connections:
- net GND is gone; now on net GNDD: U1.18 (GND), U1.35 (GND), U1.42 (GND), U1.5 (GNDANA)
- net GNDA: now also J5.3 (Pin_3); no longer C1.1, C2.1, J5.2 (Pin_2)
- net GNDD: now also C1.1, C2.1, J5.2 (Pin_2); no longer J5.3 (Pin_3)
- net SWCLK: now also J1.4 (PGD/ICSPDAT); no longer J1.5 (PGC/ICSPCLK)
- net SWDIO: now also J1.5 (PGC/ICSPCLK); no longer J1.4 (PGD/ICSPDAT)

Commit message: IO Board v3
Parts:
- removed H1, H2, H3, H4: MountingHole_Pad, MountingHole:MountingHole_3.2mm_M3_ISO7380_Pad, symbol Mechanical:MountingHole_Pad
- removed J9: Conn_01x03_Pin, Connector_PinHeader_2.54mm:PinHeader_1x03_P2.54mm_Vertical, symbol Connector:Conn_01x03_Pin
- removed U4, U5, U8: ~, custom_lib:4mm_banana_female, symbol custom_lib:4mm_female_banana
- added J11: Conn_01x04_Pin, Connector_PinHeader_2.54mm:PinHeader_1x04_P2.54mm_Vertical, symbol Connector:Conn_01x04_Pin
- added J13 (x3): Eurorack_Mono_Jack, winterbloom:AudioJack_WQP518MA, symbol winterbloom:Eurorack_Mono_Jack
Connections:
- net ADC_in: now also J11.3 (Pin_3)
- net Audio_out: now also J13.T (Tip)
- net DAC_out: now also J11.4 (Pin_4)
- net GNDA: now also U3.4 (V-), U9.4 (V-), J13.S (Sleeve), J13.S (Sleeve), J13.S (Sleeve); no longer ENC0.C, ENC1.C, ENC2.C, ENC3.C
- net GNDD: now also ENC0.C, ENC1.C, ENC2.C, ENC3.C; no longer U3.4 (V-), U9.4 (V-)
- net SCL: now also J11.1 (Pin_1)
- net SDA: now also J11.2 (Pin_2)
- net at S2.1: now also J13.T (Tip)
- net at S2.3: now also J13.T (Tip)
Other:
- note removed: "Mounting Holes"
- moved on the sheet: J5

Commit message: added IO Board dimensions
Other:
- company: (none) -> Chameleon Engine 2023
- title: (none) -> I/O Board 
Changed lines of the file:
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@@
 (kicad_sch (version 20230121) (generator eeschema)
   (paper "A3")
+  (title_block
+    (title "I/O Board ")
+    (rev "V3")
+    (company "Chameleon Engine 2023")
+  )
   (junction (at 113.03 63.5) (diameter 0) (color 0 0 0 0)
   )
