File: IOBoard_ATSAMD21/_autosave-IOBoard_ATSAMD21.kicad_sch (KiCad schematic)
At the start: 36 parts, among them J1 Conn_PIC_ICSP_ICD, J2 Conn_01x04_Male, SW1 EG_1218, SW2 EG_1218, SW3 EG_1218, SW4 EG_1218, U1 ATSAMD21G18A-A, U2 AP2112K-3.3

Commit message: updating lab PC
Parts:
- ENC0, ENC1, ENC2, ENC3: footprint Rotary_Encoder:RotaryEncoder_Bourns_Vertical_PEC12R-3xxxF-Sxxxx -> custom_lib:PEC12R-3217F-S0024-ND
Connections:
- net +3.3V: no longer SW1.1, SW2.1, SW3.1, SW4.1
- net GND: now also SW1.1, SW2.1, SW3.1, SW4.1
Changed lines of the file:
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@@
     (pin "2")
-  )
-  (symbol (lib_id "power:+3.3V") (at 110.49 99.06 0) (unit 1)
-    (in_bom yes) (on_board yes) (fields_autoplaced)
-    (property "Reference" "#PWR0111" (id 0) (at 110.49 102.87 0)
-      (effects (font (size 1.27 1.27)) hide)
-    )
-    (property "Value" "+3.3V" (id 1) (at 110.49 93.98 0))
-    (property "Footprint" "" (id 2) (at 110.49 99.06 0)
-      (effects (font (size 1.27 1.27)) hide)
-    )
-    (property "Datasheet" "" (id 3) (at 110.49 99.06 0)
-      (effects (font (size 1.27 1.27)) hide)
-    )
-    (pin "1")
   )
   (symbol (lib_id "power:PWR_FLAG") (at 166.37 187.96 0) (unit 1)
@@
     (property "Reference" "ENC2" (id 0) (at 180.34 59.69 0))
     (property "Value" "RotaryEncoder_Switch" (id 1) (at 180.34 62.23 0))
-    (property "Footprint" "Rotary_Encoder:RotaryEncoder_Bourns_Vertical_PEC12R-3xxxF-Sxxxx" (id 2) (at 176.53 65.786 0)
+    (property "Footprint" "custom_lib:PEC12R-3217F-S0024-ND" (id 2) (at 176.53 65.786 0)
       (effects (font (size 1.27 1.27)) hide)
     )
@@
     )
     (property "Datasheet" "" (id 3) (at 255.27 50.8 0)
+      (effects (font (size 1.27 1.27)) hide)
+    )
+    (pin "1")
+  )
+  (symbol (lib_id "power:GND") (at 110.49 99.06 180) (unit 1)
+    (in_bom yes) (on_board yes) (fields_autoplaced)
+    (property "Reference" "#PWR0111" (id 0) (at 110.49 92.71 0)
+      (effects (font (size 1.27 1.27)) hide)
+    )
+    (property "Value" "GND" (id 1) (at 110.49 93.98 0))
+    (property "Footprint" "" (id 2) (at 110.49 99.06 0)
+      (effects (font (size 1.27 1.27)) hide)
+    )
+    (property "Datasheet" "" (id 3) (at 110.49 99.06 0)
       (effects (font (size 1.27 1.27)) hide)
     )
@@
     (property "Reference" "ENC0" (id 0) (at 180.34 16.51 0))
     (property "Value" "RotaryEncoder_Switch" (id 1) (at 180.34 19.05 0))
-    (property "Footprint" "Rotary_Encoder:RotaryEncoder_Bourns_Vertical_PEC12R-3xxxF-Sxxxx" (id 2) (at 176.53 22.606 0)
+    (property "Footprint" "custom_lib:PEC12R-3217F-S0024-ND" (id 2) (at 176.53 22.606 0)
       (effects (font (size 1.27 1.27)) hide)
     )
@@
     (property "Reference" "ENC3" (id 0) (at 180.34 82.55 0))
     (property "Value" "RotaryEncoder_Switch" (id 1) (at 180.34 85.09 0))
-    (property "Footprint" "Rotary_Encoder:RotaryEncoder_Bourns_Vertical_PEC12R-3xxxF-Sxxxx" (id 2) (at 176.53 88.646 0)
+    (property "Footprint" "custom_lib:PEC12R-3217F-S0024-ND" (id 2) (at 176.53 88.646 0)
       (effects (font (size 1.27 1.27)) hide)
     )
@@
     (property "Reference" "ENC1" (id 0) (at 180.34 38.1 0))
     (property "Value" "RotaryEncoder_Switch" (id 1) (at 180.34 40.64 0))
-    (property "Footprint" "Rotary_Encoder:RotaryEncoder_Bourns_Vertical_PEC12R-3xxxF-Sxxxx" (id 2) (at 176.53 44.196 0)
+    (property "Footprint" "custom_lib:PEC12R-3217F-S0024-ND" (id 2) (at 176.53 44.196 0)
       (effects (font (size 1.27 1.27)) hide)
     )
@@
       (reference "#PWR0110") (unit 1) (value "+3.3V") (footprint "")
     )
-    (path "/2b549224-0b4e-476a-a384-1c3a815199ce"
-      (reference "#PWR0111") (unit 1) (value "+3.3V") (footprint "")
+    (path "/7b088d3b-84f4-478a-807f-0992a47a1908"
+      (reference "#PWR0111") (unit 1) (value "GND") (footprint "")
     )
     (path "/8364a51f-522a-4045-97f1-bb89d3186792"
@@
     )
     (path "/9500eb1b-1d42-4f52-8d28-d1067669f5e8"
-      (reference "ENC0") (unit 1) (value "RotaryEncoder_Switch") (footprint "Rotary_Encoder:RotaryEncoder_Bourns_Vertical_PEC12R-3xxxF-Sxxxx")
+      (reference "ENC0") (unit 1) (value "RotaryEncoder_Switch") (footprint "custom_lib:PEC12R-3217F-S0024-ND")
     )
     (path "/fa7625d7-e853-4b9e-a949-77e9fabc4999"
-      (reference "ENC1") (unit 1) (value "RotaryEncoder_Switch") (footprint "Rotary_Encoder:RotaryEncoder_Bourns_Vertical_PEC12R-3xxxF-Sxxxx")
+      (reference "ENC1") (unit 1) (value "RotaryEncoder_Switch") (footprint "custom_lib:PEC12R-3217F-S0024-ND")
     )
     (path "/72c889e8-7492-4719-84d0-7f508e81f71b"
-      (reference "ENC2") (unit 1) (value "RotaryEncoder_Switch") (footprint "Rotary_Encoder:RotaryEncoder_Bourns_Vertical_PEC12R-3xxxF-Sxxxx")
+      (reference "ENC2") (unit 1) (value "RotaryEncoder_Switch") (footprint "custom_lib:PEC12R-3217F-S0024-ND")
     )
     (path "/b6674150-4bc6-405d-9f7f-6bd360f25813"
-      (reference "ENC3") (unit 1) (value "RotaryEncoder_Switch") (footprint "Rotary_Encoder:RotaryEncoder_Bourns_Vertical_PEC12R-3xxxF-Sxxxx")
+      (reference "ENC3") (unit 1) (value "RotaryEncoder_Switch") (footprint "custom_lib:PEC12R-3217F-S0024-ND")
     )
     (path "/c38d78cd-b461-4746-a770-89b919ea079e"
