File: PCM5242/PCM5242.kicad_pcb (KiCad board)
At the start: 2 copper layers, 79.9 x 59.9 mm, 39 parts, among them IC1 NCP163ASN330T1G, IC2 NCP163ASN330T1G, J1 Conn_01x04_Male, J2 Conn_01x12_Male, J3 d, U1 PCM5242, Y1 ASE-24.000MHZ-ET

Commit message: DAC 3.0 V1
Parts:
- removed C11, C12: 1000pF, Capacitor_SMD:C_0603_1608Metric_Pad1.08x0.95mm_HandSolder
- removed R10, R11: 806, Resistor_SMD:R_1206_3216Metric_Pad1.30x1.75mm_HandSolder
- removed R2, R3, R4, R5, R6, R7, R8, R9: 402, Resistor_SMD:R_1206_3216Metric_Pad1.30x1.75mm_HandSolder
Connections:
- net /A10 renamed /ADR2
- net /A11 renamed /GPIO6
- net /A12 renamed /BCK
- net /A13 renamed /DIN
- net /A14 renamed /LRCK
- net /A15 renamed /ADR1
- net /A5 renamed /SDA
- net /A6 renamed /SCL
- net /A7 renamed /GPIO5
- net /A8 renamed /GPIO4
- net /A9 renamed /GPIO3
- J1 pad 1: /A1 -> /OUTLP
- J1 pad 2: /A2 -> /OUTLN
- J1 pad 3: /A3 -> /OUTRN
- J1 pad 4: /A4 -> /OUTRP
- U1 pad 10: Net-(R4-Pad1) -> /OUTLP
- U1 pad 11: Net-(R3-Pad1) -> /OUTLN
- U1 pad 12: Net-(R5-Pad1) -> /OUTRN
- U1 pad 13: Net-(R2-Pad1) -> /OUTRP
Routing:
- net /OUTRP: track 0.00 -> 33.9 mm
- net /OUTLP: track 0.00 -> 33.9 mm
- net /OUTRN: track 0.00 -> 33.0 mm
- net /OUTLN: track 0.00 -> 33.0 mm
- net /A2: track 13.1 -> 0.00 mm
- net Net-(R4-Pad1): track 13.0 -> 0.00 mm
- net Net-(R5-Pad1): track 12.2 -> 0.00 mm
- net Net-(R2-Pad1): track 11.7 -> 0.00 mm
- net Net-(R3-Pad1): track 11.3 -> 0.00 mm
- net /A3: track 10.5 -> 0.00 mm
- net Net-(C11-Pad1): track 9.18 -> 0.00 mm
- net Net-(C12-Pad1): track 9.14 -> 0.00 mm
- net Net-(C11-Pad2): track 8.92 -> 0.00 mm
- net /A4: track 8.88 -> 0.00 mm
- net /A1: track 8.57 -> 0.00 mm
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Other:
- board text added: "Analog Out"
- board text added: "Digital In"
- board text added: "University of Washington Engine 2023 Chameleon DAC - PCM5242 V.3.0 James 3/28/23"
- board text removed: "A1"
- board text removed: "A10"
- board text removed: "A11"
- board text removed: "A12"
- board text removed: "A13"
- board text removed: "A14"
- board text removed: "A15"
- board text removed: "A2"
- board text removed: "A3"
- board text removed: "A4"
- board text removed: "A5"
- board text removed: "A6"
- board text removed: "A7"
- board text removed: "A8"
- board text removed: "A9"
- board text removed: "Analog In"
- board text removed: "Digital Out"
- board text removed: "University of Washington Engine 2023 Chameleon DAC - PCM5242 V.2.1 Julian James 2/28/23"
