File: PCM5242/PCM5242.kicad_sch (KiCad schematic)
At the start: 35 parts, among them IC1 NCP163ASN330T1G, IC2 NCP163ASN330T1G, J1 Conn_01x04_Male, J2 Conn_01x12_Male, J3 d, U1 PCM5242, Y1 ASE-24.000MHZ-ET

Commit message: DAC 3.0 V1
Parts:
- removed C11, C12: 1000pF, Capacitor_SMD:C_0603_1608Metric_Pad1.08x0.95mm_HandSolder, symbol Device:C
- removed R10, R11: 806, Resistor_SMD:R_1206_3216Metric_Pad1.30x1.75mm_HandSolder, symbol Device:R
- removed R2, R3, R4, R5, R6, R7, R8, R9: 402, Resistor_SMD:R_1206_3216Metric_Pad1.30x1.75mm_HandSolder, symbol Device:R
Connections:
- net A1 is gone; now on net OUTLP: J1.1 (Pin_1)
- net A2 is gone; now on net OUTLN: J1.2 (Pin_2)
- net A3 is gone; now on net OUTRN: J1.3 (Pin_3)
- net A4 is gone; now on net OUTRP: J1.4 (Pin_4)
- net OUTRP: now reaches U1.13 (OUTRP)
- net OUTRN: now reaches U1.12 (OUTRN)
- net OUTLP: now reaches U1.10 (OUTLP)
- net OUTLN: now reaches U1.11 (OUTLN)
- net A10 renamed ADR2
- net A11 renamed GPIO6
- net A12 renamed BCK
- net A13 renamed DIN
- net A14 renamed LRCK
- net A15 renamed ADR1
- net A5 renamed SDA
- net A6 renamed SCL
- net A7 renamed GPIO5
- net A8 renamed GPIO4
- net A9 renamed GPIO3
Other:
- note added: "3.0"
- note added: "3/28/23"
- note removed: "2.1"
- note removed: "3/7/23"
- note removed: "Digital Out"
- moved on the sheet: C10, C13, C14, C15, C16, C17, C18, C19, C9, IC1, IC2, J1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
