File: PCM1863/PCM1863.kicad_pcb (KiCad board)
At the start: 2 copper layers, 60.8 x 138.6 mm, 68 parts, among them IC1 SN74AUC1G126DCKR, IC2 NCP163ASN330T1G, IC3 NCP163ASN330T1G, IC4 TXB0101DBVT, J1 Conn_01x02_Male, J10 Conn_01x10_Male, J2 Conn_01x02_Male, J3 Conn_01x02_Male, J4 USB_B_Micro, J5 Conn_01x02_Male, J6 Conn_01x02_Male, J7 Conn_01x02_Male, J8 Conn_01x10_Male, J9 Conn_01x10_Male, U1 PCM1863, Y1 ASE-24.000MHZ-ET, Y2 ASE-22.000MHZ-ET

Commit message: temp
Parts:
- removed J2, J3, J5, J6, J7: Conn_01x02_Male, Connector_PinHeader_2.54mm:PinHeader_1x02_P2.54mm_Vertical
- added R9: 4.99k, Resistor_SMD:R_0603_1608Metric_Pad0.98x0.95mm_HandSolder, F.Cu at (55.6, 31.5)
- J1: value Conn_01x02_Male -> Conn_02x05_Row_Letter_First; footprint Connector_PinHeader_2.54mm:PinHeader_1x02_P2.54mm_Vertical -> Connector_PinHeader_2.54mm:PinHeader_2x05_P2.54mm_Vertical
- moved J8 179.4 mm to (24.4, 17.5), turned to 0 degrees
- moved H4 159.0 mm to (160.0, 27.9)
- moved C4 143.0 mm to (38.2, 24.0), turned to 0 degrees
- moved J9 142.4 mm to (29.0, 17.5)
- moved C9 130.2 mm to (38.2, 36.5), turned to 0 degrees
- moved C20 128.9 mm to (46.9, 18.9), turned to 0 degrees
- moved C21 128.0 mm to (46.9, 21.4), turned to 0 degrees
- moved IC2 127.3 mm to (33.4, 44.9)
- moved C22 123.9 mm to (46.9, 24.0), turned to 0 degrees
- moved C23 123.5 mm to (46.9, 26.5), turned to 0 degrees
- moved C30 122.7 mm to (51.2, 21.4), turned to 0 degrees
- moved R2 121.6 mm to (51.2, 36.5), turned to 0 degrees
- moved R3 121.4 mm to (55.6, 16.4), turned to 0 degrees
- moved R5 120.2 mm to (55.6, 21.4), turned to 0 degrees
- moved C26 119.0 mm to (46.9, 34.0), turned to 0 degrees
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Connections:
- C11 pad 2: /VREF -> /VREF_gnd
- C14 pad 1: Net-(C14-Pad1) -> +1V8
- C16 pad 1: Net-(C14-Pad1) -> +1V8
- C2 pad 1: /XO -> /XO_gnd
- C3 pad 2: /XI -> /XI_gnd
- C7 pad 1: Net-(C14-Pad1) -> +1V8
- D1 pad 2: Net-(C14-Pad1) -> +1V8
- IC1 pad 1: GNDD -> /XI_EN
- IC4 pad 5: Net-(IC4-Pad5) -> /XO_EN
- J1 pad 1: GNDD -> (no net)
- J1 pad 2: Net-(IC4-Pad5) -> (no net)
- R23 pad 2: Net-(IC4-Pad5) -> /XO_EN
- U1 pad 10: Net-(U1-Pad10) -> /XI
- U1 pad 11: Net-(C14-Pad1) -> +1V8
- U1 pad 6: Net-(U1-Pad6) -> /VREF
- U1 pad 9: Net-(U1-Pad9) -> /XO
Routing:
- net +3V3: track 79.2 -> 0.00 mm
- net +1V8: track 68.2 -> 0.00 mm
- net VCC: track 64.4 -> 0.00 mm
- net /SCKI(3.3V): track 61.4 -> 0.00 mm
- net /MD4/MISO/GPIO0: track 58.1 -> 0.00 mm
- net /MD5/GPIO1/INTA/DMIN: track 57.1 -> 0.00 mm
- net /INT/GPIO3/INTC: track 56.7 -> 0.00 mm
- net /MD6/GPIO2/INTB/DMCLK: track 56.3 -> 0.00 mm
- net /DOUT: track 56.3 -> 0.00 mm
- net /BCK: track 55.9 -> 0.00 mm
- net /LRCK: track 55.4 -> 0.00 mm
- net /XI: track 54.1 -> 0.00 mm
- net GNDD: track 53.2 -> 0.00 mm, vias 31 -> 0
- net /OSC: track 47.3 -> 0.00 mm, vias 2 -> 0
- net /DOUT2/MD2/MOSI/SDA: track 46.6 -> 0.00 mm
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- removed copper zone on F.Cu, net +3.3VA
- removed copper zone on F.Cu, net +3V3
- removed copper zone on B.Cu, net GNDA
- removed copper zone on F.Cu, net GNDA
- removed copper zone on B.Cu, net GNDD
- removed copper zone on F.Cu, net GNDD
- removed copper zone on F.Cu, net VCC
Other:
- board size 60.8 x 138.6 mm -> 76.2 x 128.5 mm
- board text removed: "+1.8V"
- board text removed: "+3.3V"
- board text removed: "+3.3VA"
- board text removed: "+3.3VA_ON"
- board text removed: "+3.3V_ON"
- board text removed: "22MHz"
- board text removed: "24MHz"
- board text removed: "AD"
- board text removed: "ADC"
- board text removed: "Analog"
- board text removed: "BCK"
- board text removed: "DOUT"
- board text removed: "Digital"
- board text removed: "GNDA"
- board text removed: "GNDD"
- board text removed: "GPIO0"
- board text removed: "GPIO1"
- board text removed: "GPIO2"
- board text removed: "GPIO3"
- board text removed: "IN1"
- board text removed: "IN2"
- board text removed: "IN3"
- board text removed: "IN4"
- board text removed: "LDO_CONN"
- board text removed: "LDO_ON"
- board text removed: "LRCK"
- board text removed: "MD0"
- board text removed: "OSC"
- board text removed: "SCKI(3.3V)"
- board text removed: "SCL"
- board text removed: "SDA"
- board text removed: "University of Washington Engine 2023 - Chameleon ADC - PCM1863 v.5 Ford 03/12/2023"
- board text removed: "VCC"
- board text removed: "VCC_IN"
- board text removed: "VCC_ON"
- board text removed: "VREF"
- board text removed: "VREF_CONN"
- board text removed: "XI"
- board text removed: "XI_BUFF"
- board text removed: "XI_CONN"
- board text removed: "XI_TO_GND"
- board text removed: "XO"
- board text removed: "XO_BUFF"
- board text removed: "XO_CONN"
- board text removed: "XO_EN"

Commit message: adc v6
Parts:
- removed C11: 1uF, Capacitor_SMD:C_0603_1608Metric_Pad1.08x0.95mm_HandSolder
- removed C2, C3: 20pF, Capacitor_SMD:C_0603_1608Metric_Pad1.08x0.95mm_HandSolder
- removed J10, J9: Conn_01x10_Male, Connector_PinHeader_2.54mm:PinHeader_1x10_P2.54mm_Vertical
- added C34: 20pF, Capacitor_SMD:C_0603_1608Metric_Pad1.08x0.95mm_HandSolder, F.Cu at (100.6, 34.3)
- added C35: 20pF, Capacitor_SMD:C_0603_1608Metric_Pad1.08x0.95mm_HandSolder, F.Cu at (111.5, 34.4)
- added C36: 1uF, Capacitor_SMD:C_0603_1608Metric_Pad1.08x0.95mm_HandSolder, F.Cu at (104.1, 34.3)
- added G***: LOGO, LOGO, F.Cu at (128.5, 39.6)
- added G***: LOGO, LOGO, F.Cu at (138.7, 128.5)
- added J11: Conn_01x04_Pin, Connector_PinHeader_2.54mm:PinHeader_1x04_P2.54mm_Vertical, F.Cu at (158.5, 80.2)
- added J2: Conn_01x03_Pin, Connector_PinHeader_2.54mm:PinHeader_1x03_P2.54mm_Vertical, F.Cu at (158.5, 95.5)
- added J3: Conn_01x04_Pin, Connector_PinHeader_2.54mm:PinHeader_1x04_P2.54mm_Vertical, F.Cu at (158.5, 66.3)
- added J5: Conn_01x04_Pin, Connector_PinHeader_2.54mm:PinHeader_1x04_P2.54mm_Vertical, F.Cu at (143.8, 29.4)
- added J6: Conn_01x10_Pin, Connector_PinHeader_2.54mm:PinHeader_1x10_P2.54mm_Vertical, F.Cu at (98.8, 54.3)
- added J7: Conn_01x05_Pin, Connector_PinHeader_2.54mm:PinHeader_1x05_P2.54mm_Vertical, F.Cu at (116.1, 90.1)
- J1: value Conn_02x05_Row_Letter_First -> Conn_01x04_Pin; footprint Connector_PinHeader_2.54mm:PinHeader_2x05_P2.54mm_Vertical -> Connector_PinHeader_2.54mm:PinHeader_1x04_P2.54mm_Vertical
- J8: value Conn_01x10_Male -> Conn_02x05_Top_Bottom; footprint Connector_PinHeader_2.54mm:PinHeader_1x10_P2.54mm_Vertical -> Connector_PinHeader_2.54mm:PinHeader_2x05_P2.54mm_Vertical
- moved C4 147.5 mm to (122.0, 145.3), turned to -90 degrees
- moved C6 143.9 mm to (129.0, 140.6), turned to 180 degrees
- moved R2 138.2 mm to (134.1, 147.1), turned to 90 degrees
- moved IC2 137.3 mm to (127.0, 145.3)
- moved C9 135.8 mm to (119.4, 145.3), turned to -90 degrees
- moved D2 131.8 mm to (131.6, 147.1), turned to 90 degrees
- moved R4 129.5 mm to (105.1, 138.7), turned to 180 degrees
- moved C22 118.4 mm to (160.7, 56.6), turned to 180 degrees
- moved R3 117.7 mm to (99.9, 125.5)
- moved U1 117.1 mm to (141.7, 67.8)
- moved C30 115.9 mm to (160.6, 59.7), turned to 180 degrees
- moved C25 115.7 mm to (105.8, 131.0), turned to 180 degrees
- moved C24 115.7 mm to (105.8, 128.5), turned to 180 degrees
- moved C1 115.6 mm to (133.6, 81.8), turned to -90 degrees
- moved C5 114.4 mm to (103.9, 120.1)
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Connections:
- H1 pad 1: GNDD -> GNDA
- H2 pad 1: GNDA -> GNDD
- H3 pad 1: GNDA -> GNDD
- H4 pad 1: GNDD -> GNDA
- IC1 pad 1: /XI_EN -> /XI_DIS
- IC4 pad 5: /XO_EN -> /XO_DIS
- J1 pad 1: (no net) -> /VIN1P
- J1 pad 2: (no net) -> /VIN2P
- J1 pad 3: (no net) -> /VIN3P
- J1 pad 4: (no net) -> /VIN4P
- J8 pad 1: GNDA -> /XO
- J8 pad 10: /SCKI(3.3V) -> /XI_gnd
- J8 pad 2: GNDA -> /XO_gnd
- J8 pad 3: /MD4/MISO/GPIO0 -> /VREF
- J8 pad 4: /MD5/GPIO1/INTA/DMIN -> /VREF_gnd
- J8 pad 5: /MD6/GPIO2/INTB/DMCLK -> /XO_DIS
- J8 pad 6: /INT/GPIO3/INTC -> GNDD
- J8 pad 7: /DOUT -> /XI_DIS
- J8 pad 8: /BCK -> GNDD
- J8 pad 9: /LRCK -> /XI
- R23 pad 2: /XO_EN -> /XO_DIS
- R9 pad 2: /XI_EN -> /XI_DIS
Routing:
- net GNDD: track 0.00 -> 149.3 mm, vias 0 -> 20
- net +3.3VA: track 0.00 -> 96.2 mm, vias 0 -> 2
- net /XO: track 0.00 -> 94.1 mm, vias 0 -> 1
- net /VREF: track 0.00 -> 71.8 mm
- net /XI: track 0.00 -> 71.4 mm, vias 0 -> 3
- net VCC: track 0.00 -> 62.2 mm
- net +1V8: track 0.00 -> 58.4 mm, vias 0 -> 2
- net +3V3: track 0.00 -> 48.0 mm
- net /XO_BUFF: track 0.00 -> 44.8 mm, vias 0 -> 1
- net /BCK: track 0.00 -> 38.1 mm
- net /SCKI(3.3V): track 0.00 -> 35.4 mm, vias 0 -> 1
- net /XI_DIS: track 0.00 -> 33.7 mm, vias 0 -> 2
- net GNDA: track 0.00 -> 33.2 mm, vias 0 -> 72
- net /LRCK: track 0.00 -> 32.8 mm
- net /DOUT: track 0.00 -> 31.5 mm
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- added copper zone on F.Cu, net +3.3VA
- added copper zone on F.Cu, net +3V3
- added copper zone on B.Cu, net GNDA
- added copper zone on F.Cu, net GNDA
- added copper zone on B.Cu, net GNDD
- added copper zone on F.Cu, net GNDD
- added copper zone on F.Cu, net VCC
Other:
- outline, holes or cut-outs redrawn
- board text added: "AD"
- board text added: "ADC - PCM1863 v.6 Nathan Ford 04/14/2023"
- board text added: "ADC Clocks"
- board text added: "AVDD"
- board text added: "AVDD (+3.3VA)"
- board text added: "Artwork by: Trina Kha"
- board text added: "BCK"
- board text added: "DOUT"
- board text added: "DVDD"
- board text added: "DVDD (+3.3V)"
- board text added: "Enable/ Disable"
- board text added: "GNDA"
- board text added: "GNDD"
- board text added: "GPIO"
- board text added: "GPIO0"
- board text added: "GPIO1"
- board text added: "GPIO2"
- board text added: "GPIO3"
- board text added: "I2C"
- board text added: "I2S"
- board text added: "IN1"
- board text added: "IN2"
- board text added: "IN3"
- board text added: "IN4"
- board text added: "Inputs [0V, +5V]"
- board text added: "LDO"
- board text added: "LRCK"
- board text added: "MDO"
- board text added: "OSC"
- board text added: "OUT"
- board text added: "Power"
- board text added: "SCKI(3.3V)"
- board text added: "SCL"
- board text added: "SDA"
- board text added: "Test Points"
- board text added: "University of Washington ENGINE 2023 - Chameleon"
- board text added: "VCC"
- board text added: "VCC (+5V)"
- board text added: "VIN1P"
- board text added: "VIN2P"
- board text added: "VIN3P"
- board text added: "VINP4"
- board text added: "VREF"
- board text added: "VREF_ENABLE"
- board text added: "XI"
- board text added: "XI_DISABLE"
- board text added: "XI_POWER_OFF"
- board text added: "XO"
- board text added: "XO_BUFF"
- board text added: "XO_DIS"
- board text added: "XO_POWER_OFF"

Commit message: adc v6
Other:
- board text added: "22MHz"
- board text added: "24MHz"
- board text added: "XI_BUFF"
Changed lines of the file:
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@@
     (property "ki_description" "TXB0101DBVT")
     (attr smd)
-    (fp_text reference "IC4" (at -0.762 2.794) (layer "F.SilkS")
+    (fp_text reference "IC4" (at -0.762 2.794) (layer "F.SilkS") hide
         (effects (font (size 1.27 1.27) (thickness 0.254)))
     )
@@
     (property "ki_description" "ABRACON - ASE-24.000MHZ-ET - Oscillator, 24 MHz, 100 ppm, SMD, 3.2mm x 2.5mm, LVCMOS, 3.3 V, ASE Series")
     (attr smd)
-    (fp_text reference "Y1" (at 1.778 3.556) (layer "F.SilkS")
+    (fp_text reference "Y1" (at 1.778 3.556) (layer "F.SilkS") hide
         (effects (font (size 1.27 1.27) (thickness 0.254)))
     )
@@
     (property "ki_description" "Single Bus Buffer Gate With 3-State Output")
     (attr smd)
-    (fp_text reference "IC1" (at -0.5225 2.54) (layer "F.SilkS")
+    (fp_text reference "IC1" (at -0.5225 2.54) (layer "F.SilkS") hide
         (effects (font (size 1.27 1.27) (thickness 0.254)))
     )
@@
     (property "ki_description" "ABRACON - ASE-24.000MHZ-ET - Oscillator, 24 MHz, 100 ppm, SMD, 3.2mm x 2.5mm, LVCMOS, 3.3 V, ASE Series")
     (attr smd)
-    (fp_text reference "Y2" (at -2.5545 -3.556) (layer "F.SilkS")
+    (fp_text reference "Y2" (at -2.5545 -3.556) (layer "F.SilkS") hide
         (effects (font (size 1.27 1.27) (thickness 0.254)))
     )
@@
     (effects (font (size 1 1) (thickness 0.153)) (justify left bottom))
   )
+  (gr_text "XO_BUFF" (at 117.348 60.936) (layer "F.SilkS")
+    (effects (font (size 1 1) (thickness 0.153)) (justify left bottom))
+  )
   (gr_text "LRCK" (at 161.29 98.528) (layer "F.SilkS")
     (effects (font (size 1 1) (thickness 0.153)) (justify left bottom))
@@
     (effects (font (size 1 1) (thickness 0.153)) (justify right bottom))
   )
+  (gr_text "24MHz" (at 137.16 79.478) (layer "F.SilkS")
+    (effects (font (size 1 1) (thickness 0.153)) (justify left bottom))
+  )
   (gr_text "Power" (at 92.71 80.748) (layer "F.SilkS")
     (effects (font (size 1.5 1.5) (thickness 0.2295)) (justify left top))
@@
     (effects (font (size 1 1) (thickness 0.153)) (justify right bottom))
   )
+  (gr_text "22MHz" (at 105.918 69.318) (layer "F.SilkS")
+    (effects (font (size 1 1) (thickness 0.153)) (justify left bottom))
+  )
   (gr_text "VCC (+5V)" (at 92.71 135.358) (layer "F.SilkS")
     (effects (font (size 1.5 1.5) (thickness 0.2295)) (justify left bottom))
@@
     (effects (font (size 1 1) (thickness 0.153)) (justify left bottom))
   )
+  (gr_text "XI_BUFF" (at 115.316 73.89) (layer "F.SilkS")
+    (effects (font (size 1 1) (thickness 0.153)) (justify left bottom))
+  )

Commit message: plz work
Parts:
- removed C17: .01uF, Capacitor_SMD:C_0603_1608Metric_Pad1.08x0.95mm_HandSolder
- removed C19: 2.2uF, Capacitor_SMD:C_0603_1608Metric_Pad1.08x0.95mm_HandSolder
- removed C20, C23, C27, C32: 0.01uF, Capacitor_SMD:C_0603_1608Metric_Pad1.08x0.95mm_HandSolder
- removed C21, C26, C31, C33: 10uF, Capacitor_SMD:C_0603_1608Metric_Pad1.08x0.95mm_HandSolder
- removed C28, C29: 0.1uF, Capacitor_SMD:C_0603_1608Metric_Pad1.08x0.95mm_HandSolder
- removed C34, C35: 20pF, Capacitor_SMD:C_0603_1608Metric_Pad1.08x0.95mm_HandSolder
- removed C36: 1uF, Capacitor_SMD:C_0603_1608Metric_Pad1.08x0.95mm_HandSolder
- removed the G*** at (128.5, 39.6)
- removed the G*** at (138.7, 128.5)
- removed H1, H2, H3, H4: MountingHole_Pad, MountingHole:MountingHole_3.2mm_M3_Pad
- removed IC1: SN74AUC1G126DCKR, custom_lib:SOT65P210X110-5N
- removed IC4: TXB0101DBVT, custom_lib:SOT95P280X145-6N
- removed J11, J5: Conn_01x04_Pin, Connector_PinHeader_2.54mm:PinHeader_1x04_P2.54mm_Vertical
- removed J7: Conn_01x05_Pin, Connector_PinHeader_2.54mm:PinHeader_1x05_P2.54mm_Vertical
- removed J8: Conn_02x05_Top_Bottom, Connector_PinHeader_2.54mm:PinHeader_2x05_P2.54mm_Vertical
- removed R23: 4.99k, Resistor_SMD:R_0603_1608Metric_Pad0.98x0.95mm_HandSolder
- removed R5, R6, R7, R8: 100, Resistor_SMD:R_0603_1608Metric_Pad0.98x0.95mm_HandSolder
- removed Y2: ASE-22.000MHZ-ET, custom_lib:ASE24000MHZET
- added C2: 2.2uF, Capacitor_SMD:C_0603_1608Metric_Pad1.08x0.95mm_HandSolder, F.Cu at (211.2, 41.0)
- added C3: 2.2uF, Capacitor_SMD:C_0603_1608Metric_Pad1.08x0.95mm_HandSolder, F.Cu at (211.2, 38.5)
- added G***: LOGO, custom_lib:uw_chameleon, F.Cu at (210.8, 125.3)
- added G***: LOGO, custom_lib:uw_chameleon, F.Cu at (175.9, 125.3)
- added G***: LOGO, custom_lib:blank_chameleon, F.Cu at (192.4, 86.0)
- added R10: 100k, Resistor_SMD:R_0603_1608Metric_Pad0.98x0.95mm_HandSolder, F.Cu at (176.9, 54.5)
- added R11: 100k, Resistor_SMD:R_0603_1608Metric_Pad0.98x0.95mm_HandSolder, F.Cu at (179.5, 58.6)
- added R12: 100k, Resistor_SMD:R_0603_1608Metric_Pad0.98x0.95mm_HandSolder, F.Cu at (182.0, 58.6)
- J2: value Conn_01x03_Pin -> Conn_01x04_Pin; footprint Connector_PinHeader_2.54mm:PinHeader_1x03_P2.54mm_Vertical -> Connector_PinHeader_2.54mm:PinHeader_1x04_P2.54mm_Vertical
- J4: value USB_B_Micro -> Conn_01x04_Pin; footprint Connector_USB:USB_Micro-B_Wuerth_629105150521 -> Connector_PinHeader_2.54mm:PinHeader_1x04_P2.54mm_Vertical
- R9: value 4.99k -> 100k
- moved J6 131.8 mm to (203.2, 134.8), turned to -90 degrees
- moved J4 128.7 mm to (210.8, 67.5)
- moved FB1 124.9 mm to (201.5, 137.4), turned to 180 degrees
- moved C5 102.1 mm to (182.0, 54.4), turned to -90 degrees
- moved C6 89.9 mm to (182.0, 67.9), turned to -90 degrees
- moved C9 89.3 mm to (204.1, 117.1), turned to 0 degrees
- moved R4 87.8 mm to (191.8, 124.7), turned to -90 degrees
- moved C4 87.7 mm to (204.1, 114.5), turned to 0 degrees
- moved D4 87.5 mm to (191.8, 129.1), turned to -90 degrees
- moved R3 86.6 mm to (185.3, 111.0), turned to 90 degrees
- moved R2 84.8 mm to (210.9, 111.1)
- moved D2 84.8 mm to (208.3, 111.1)
- moved IC2 84.7 mm to (204.5, 111.0)
- moved D3 83.6 mm to (182.8, 111.0), turned to 90 degrees
- moved IC3 74.4 mm to (179.0, 111.0), turned to 0 degrees
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Connections:
- J1 pad 2: /VIN2P -> /VIN1M
- J1 pad 3: /VIN3P -> /VIN1P
- J1 pad 4: /VIN4P -> /VINR1
- J4 pad 1: VCC -> /MD4/MISO/GPIO0
- J4 pad 2: unconnected-(J4-D--Pad2) -> /MD5/GPIO1/INTA/DMIN
- J4 pad 3: unconnected-(J4-D+-Pad3) -> /MD6/GPIO2/INTB/DMCLK
- J4 pad 4: unconnected-(J4-ID-Pad4) -> /INT/GPIO3/INTC
- J6 pad 1: GNDA -> GNDD
- J6 pad 10: +1V8 -> +3.3VA
- J6 pad 2: /VREF -> +3V3
- J6 pad 3: GNDD -> GNDA
- J6 pad 4: +3.3VA -> /VREF
- J6 pad 6: +3V3 -> VCC
- J6 pad 8: VCC -> +1V8
- R9 pad 1: +3V3 -> GNDA
- R9 pad 2: /XI_DIS -> /VREF
- U1 pad 1: Net-(U1-VINL2/VIN1M) -> /VIN1M
- U1 pad 29: /VIN4P -> Net-(U1-VINL3/VIN4P)
- U1 pad 30: /VIN3P -> Net-(U1-VINR3/VIN3P)
- U1 pad 4: /VIN2P -> /VINR1
Routing:
- net GNDD: track 149.3 -> 15.4 mm, vias 20 -> 42
- net /XO: track 94.1 -> 14.8 mm, vias 1 -> 0
- net +3.3VA: track 96.2 -> 31.4 mm, vias 2 -> 0
- net /XI: track 71.4 -> 12.8 mm, vias 3 -> 0
- net VCC: track 62.2 -> 5.35 mm
- net /VREF: track 71.8 -> 120.3 mm, vias 0 -> 2
- net /XO_BUFF: track 44.8 -> 0.00 mm, vias 1 -> 0
- net +1V8: track 58.4 -> 101.9 mm, vias 2 -> 0
- net +3V3: track 48.0 -> 6.06 mm
- net /XI_DIS: track 33.7 -> 0.00 mm, vias 2 -> 0
- net /VIN4P: track 29.8 -> 0.00 mm
- net /OSC: track 29.7 -> 0.00 mm
- net /XO_DIS: track 29.4 -> 0.00 mm, vias 2 -> 0
- net /VIN2P: track 26.8 -> 0.00 mm
- net Net-(U1-VINR3/VIN3P): track 0.00 -> 26.1 mm
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Other:
- board size 76.2 x 128.5 mm -> 50.8 x 112 mm
- board text added: "+3.3VA LDO"
- board text added: "+3.3VD LDO"
- board text added: "24MHz Crystal"
- board text added: "3.3VA"
- board text added: "3.3VD"
- board text added: "5V"
- board text added: "ADC - PCM1863 v.7 Nathan Ford 05/19/2023"
- board text added: "Input Signals"
- board text added: "PCM1863 ADC"
- board text added: "Project Mentor: Dr. Eric Klavins"
- board text added: "SCKI"
- board text added: "SYS_CLK"
- board text added: "VIN1M"
- board text added: "VINL1"
- board text added: "VINR1"
- board text added: "[0V, +2.1V] SE [0V, +4.2V] DIFF"
- board text added: "https://github.com/ jelkinsjames/ chameleon-PCB.git"
- board text removed: "22MHz"
- board text removed: "24MHz"
- board text removed: "ADC - PCM1863 v.6 Nathan Ford 04/14/2023"
- board text removed: "ADC Clocks"
- board text removed: "AVDD"
- board text removed: "AVDD (+3.3VA)"
- board text removed: "DVDD"
- board text removed: "DVDD (+3.3V)"
- board text removed: "Enable/ Disable"
- board text removed: "IN1"
- board text removed: "IN2"
- board text removed: "IN3"
- board text removed: "IN4"
- board text removed: "Inputs [0V, +5V]"
- board text removed: "OSC"
- board text removed: "OUT"
- board text removed: "SCKI(3.3V)"
- board text removed: "Test Points"
- board text removed: "VCC"
- board text removed: "VCC (+5V)"
- board text removed: "VIN2P"
- board text removed: "VIN3P"
- board text removed: "VINP4"
- board text removed: "VREF_ENABLE"
- board text removed: "XI"
- board text removed: "XI_BUFF"
- board text removed: "XI_DISABLE"
- board text removed: "XI_POWER_OFF"
- board text removed: "XO"
- board text removed: "XO_BUFF"
- board text removed: "XO_DIS"
- board text removed: "XO_POWER_OFF"
