File: PCM1863/PCM1863.kicad_sch (KiCad schematic)
At the start: 86 parts, among them IC1 SN74AUC1G126DCKR, IC2 NCP163ASN330T1G, IC3 NCP163ASN330T1G, IC4 TXB0101DBVT, J1 Conn_01x10_Male, J2 Conn_01x10_Male, J3 Conn_01x10_Male, J4 USB_B_Micro, U1 PCM1863, Y1 ASE-24.000MHZ-ET, Y2 ASE-22.000MHZ-ET

Commit message: schematic v5
Parts:
- removed FB2, FB3, FB4, FB5, FB6: FerriteBead, Inductor_SMD:L_0603_1608Metric_Pad1.05x0.95mm_HandSolder, symbol Device:FerriteBead
- removed J1, J2, J3: Conn_01x10_Male, Connector_PinHeader_2.54mm:PinHeader_1x10_P2.54mm_Vertical, symbol Connector:Conn_01x10_Male
- removed JP1, JP10, JP11, JP2, JP3, JP4, JP6, JP8, JP9: Jumper_2_Open, custom_lib:TestPoint_Bridge_Pitch2.54mm_Drill0.7mm, symbol Jumper:Jumper_2_Open
- removed JP5, JP7: Jumper_2_Bridged, custom_lib:TestPoint_Bridge_Pitch2.54mm_Drill0.7mm, symbol Jumper:Jumper_2_Bridged
- removed R10, R11, R15, R16, R19, R20: 2.2k, Resistor_SMD:R_0603_1608Metric_Pad0.98x0.95mm_HandSolder, symbol Device:R
- removed R12, R13, R17, R18, R21, R22: 100k, Resistor_SMD:R_0603_1608Metric_Pad0.98x0.95mm_HandSolder, symbol Device:R
- added C30: 2.2uF, Capacitor_SMD:C_0603_1608Metric_Pad1.08x0.95mm_HandSolder, symbol Device:C
- added C31, C33: 10uF, Capacitor_SMD:C_0603_1608Metric_Pad1.08x0.95mm_HandSolder, symbol Device:C
- added C32: 0.01uF, Capacitor_SMD:C_0603_1608Metric_Pad1.08x0.95mm_HandSolder, symbol Device:C
- added J1, J2, J3, J5, J6, J7: Conn_01x02_Male, Connector_PinHeader_2.54mm:PinHeader_1x02_P2.54mm_Vertical, symbol Connector:Conn_01x02_Male
- added J10, J8, J9: Conn_01x10_Male, Connector_PinHeader_2.54mm:PinHeader_1x10_P2.54mm_Vertical, symbol Connector:Conn_01x10_Male
- C10, C15, C16, C28, C29: value 0.1uF-16V -> 0.1uF
- C11: value 2.2uF -> 1uF
- C12, C14, C8: value 10uF-10V -> 10uF-Tant
- C13: value 0.1uF-50V -> 0.1uF
- C18, C19, C22: value 10uF-16V -> 2.2uF
- C2, C3: value 20pF-50V -> 20pF
- C20, C23, C27: value 10uF-16V -> 0.01uF
- C21, C26: value 10uF-16V -> 10uF
- C24: value 1uF -> 0.1uF
- C25, C9: value 10uF -> 10uF-Tant
- C5: value 0.1uF -> 1uF
- H1, H2, H3, H4: footprint MountingHole:MountingHole_2.2mm_M2_Pad -> MountingHole:MountingHole_3.2mm_M3_Pad
- R1, R5, R6: value 2.2k -> 100
- R4: value 2.2k -> 10k
- R7, R8: value 100k -> 100
Connections:
- net VINL2 is gone; now on net GNDA: C27.1
- net VINL4 is gone; now on net GNDA: C23.1
- net VINR3 is gone; now on net GNDA: C20.1
- net VINR4 is gone; now on net GNDA: C22.1
- net +1V8: now also J10.9 (Pin_9), J5.1 (Pin_1); no longer C14.1, C16.1, C7.1, D1.2 (A), U1.11 (LDO)
- net +3.3VA: now also C6.2, D2.2 (A), IC2.5 (OUT), J10.7 (Pin_7); no longer C24.2, D3.2 (A), IC3.5 (OUT)
- net +3V3: now also C5.2, D3.2 (A), IC3.5 (OUT), J10.8 (Pin_8); no longer C6.2, D2.2 (A), IC2.5 (OUT)
- net BCK: now also J8.9 (Pin_9)
- net DOUT: now also J8.8 (Pin_8)
- net DOUT2/MD2/MOSI/SDA: now also J9.4 (Pin_4)
- net GNDA: now also C18.1, C19.1, C24.2, C5.1, C30.1, C32.1, J10.5 (Pin_5), J10.6 (Pin_6); no longer C24.1, C5.2, R7.1, R8.2
- net GNDD: now also C2.2, J1.1 (Pin_1), J10.2 (Pin_2), J10.3 (Pin_3), J10.4 (Pin_4), J6.2 (Pin_2); no longer C2.1
- net INT/GPIO3/INTC: now also J8.7 (Pin_7)
- net LRCK: now also J8.10 (Pin_10)
- net MD1/MS/AD: now also J9.2 (Pin_2)
- net MD3/MC/SCL: now also J9.3 (Pin_3)
- net MD4/MISO/GPIO0: now also J8.4 (Pin_4)
- net MD5/GPIO1/INTA/DMIN: now also J8.5 (Pin_5)
- net MD6/GPIO2/INTB/DMCLK: now also J8.6 (Pin_6)
- net MDO: now also J9.1 (Pin_1)
- net OSC: now also Y2.3 (OUTPUT), J8.1 (Pin_1); no longer Y1.3 (OUTPUT)
- net SCKI(3.3V): now also Y1.3 (OUTPUT), J8.3 (Pin_3); no longer Y2.3 (OUTPUT)
- net VCC: now also C24.1, J10.1 (Pin_1); no longer C5.1
- net XI: now also J2.1 (Pin_1), J6.1 (Pin_1), J9.9 (Pin_9); no longer U1.10 (XI)
- net XO: now also C2.1, IC4.3 (A), J3.2 (Pin_2), J9.10 (Pin_10); no longer C2.2, U1.9 (XO)
- net XO_BUFF: now also J8.2 (Pin_2)
- net at IC4.5 (OE), R23.2: now also J1.2 (Pin_2)
- net at U1.6 (VREF): now also J7.1 (Pin_1); no longer C11.2
- net 1L: no longer names the net of C19.2
- net 1L: now also U1.1 (VINL2/VIN1M); no longer U1.3 (VINL1/VIN1P)
- net 1R: no longer names the net of C18.2
- net 1R: now also U1.2 (VINR2/VIN2M); no longer U1.4 (VINR1/VIN2P)
- net 2L renamed VIN2P
- net VIN2P: now also R7.2, U1.4 (VINR1/VIN2P); no longer U1.1 (VINL2/VIN1M)
- net 2R renamed IN3
- net IN3: now also J9.7 (Pin_7); no longer U1.2 (VINR2/VIN2M)
- net 3L renamed IN4
- net IN4: now also J9.8 (Pin_8); no longer U1.29 (VINL3/VIN4P)
- net 3R renamed VIN3P
- net VIN3P: now also C23.2, R6.2; no longer C20.2
- net 4L: no longer names the net of U1.27 (VINL4/VIN4M)
- net 4L: now also C30.2; no longer C23.2
- net 4R: no longer names the net of C22.2, U1.28 (VINR4/VIN3M)
- net MICBIAS: no longer names the net of C13.2, U1.5 (Mic_Bias)
- net MICBIAS: no longer R5.1, R6.1
- removed net VINL1: C19.1, R5.2, R7.2
- net VINL3: no longer names the net of C21.1
- net VINL3: now also R5.1
- removed net VINR1: C18.1, R6.2, R8.1
- net VINR2: no longer names the net of C26.1
- net VINR2: now also R6.1
- new net: C14.1, C16.1, C7.1, D1.2 (A), J5.2 (Pin_2), U1.11 (LDO)
- new net: J2.2 (Pin_2), U1.10 (XI)
- new net: C33.1, R8.1
- new net: C31.1, R7.1
- new net: J3.1 (Pin_1), U1.9 (XO)
- new net IN1: C33.2, J9.5 (Pin_5)
- new net IN2: C31.2, J9.6 (Pin_6)
- new net VIN1P: C32.2, R8.2, U1.3 (VINL1/VIN1P)
- new net VIN4P: C20.2, R5.2, U1.29 (VINL3/VIN4P)
- new net VREF: C11.2, J10.10 (Pin_10), J7.2 (Pin_2)
- no-connect marks 8 -> 6
Other:
- note added: "5V"
- note added: "AD: I2C address"
- note added: "D+ and D- can be used for serial communication, but we are not"
- note added: "Digital Input and Output Pins"
- note added: "Do I want to change to digital ground because the power supply is noisy?"
- note added: "Ferrite Bead"
- note added: "GNDD is connected to GNDA with a ferrite bead(inductor) to form a common ground"
- note added: "I2C and Analog Input Pins"
- note added: "I2S bit clock"
- note added: "I2S data"
- note added: "I2S world clock"
- note added: "Input 1.8V clock"
- note added: "MD0: I2C mode select"
- note added: "Mounting Holes (M3)"
- note added: "Not used, grounded"
- note added: "Optional jump to ground"
- note added: "Optional jump to ground to disable buffer"
- note added: "Output 1.8V clock"
- note added: "Output enable (OE): High - on Low - off"
- note added: "PCM1863 Analog to Digital Converter (ADC)"
- note added: "Power and Ground Pins"
- note added: "SCL: I2C clock"
- note added: "SDA: I2C data"
- note added: "Single-Ended (SE) Inputs"
- note added: "Single-Ended (SE) input pins"
- note added: "System input clock"
- note added: "Test point or jump to ground"
- note added: "Test points: XO, XI, LDO, VREF"
- note added: "Using single-ended differential pairs. All "P"s connect to an input while all "M"s are grounded."
- note added: "Vref = AVDD / 2"
- note removed: "3.3V Analog LDO"
- note removed: "ADC1863"
- note removed: "Analog Pins"
- note removed: "Controller Pins"
- note removed: "D+ and D- can be used for serial communication"
- note removed: "Digital Pins"
- note removed: "Ferrite Beads"
- note removed: "Mounting Holes"
- note removed: "Put a surge protector connecting the positive ends of the 20pF caps"
- note removed: "To Controller or connect to GND or IOVDD"
- note removed: "VIN LR(1-4)"
- moved on the sheet: C1, C10, C11, C12, C13, C14, C15, C16, C17, C2, C28, C29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

Commit message: v5 finished
Connections:
- net +1V8: now also J10.7 (Pin_7); no longer J10.9 (Pin_9)
- net +3.3VA: now also C5.2, D3.2 (A), IC3.5 (OUT), J10.5 (Pin_5); no longer C6.2, D2.2 (A), IC2.5 (OUT), J10.7 (Pin_7)
- net +3V3: now also C6.2, D2.2 (A), IC2.5 (OUT), J10.3 (Pin_3); no longer C5.2, D3.2 (A), IC3.5 (OUT), J10.8 (Pin_8)
- net BCK: now also J8.8 (Pin_8); no longer J8.9 (Pin_9)
- net DOUT: now also J8.7 (Pin_7); no longer J8.8 (Pin_8)
- net DOUT2/MD2/MOSI/SDA: now also J9.10 (Pin_10); no longer J9.4 (Pin_4)
- net GNDA: now also H3.1, J10.2 (Pin_2), J10.8 (Pin_8), J8.1 (Pin_1), J8.2 (Pin_2), J9.1 (Pin_1); no longer H1.1, J10.5 (Pin_5), J10.6 (Pin_6)
- net GNDD: now also H1.1, J4.6 (Shield); no longer H3.1, J10.2 (Pin_2), J10.3 (Pin_3), J10.4 (Pin_4)
- net IN1: now also J9.3 (Pin_3); no longer J9.5 (Pin_5)
- net IN2: now also J9.4 (Pin_4); no longer J9.6 (Pin_6)
- net IN3: now also J9.5 (Pin_5); no longer J9.7 (Pin_7)
- net IN4: now also J9.6 (Pin_6); no longer J9.8 (Pin_8)
- net INT/GPIO3/INTC: now also J8.6 (Pin_6); no longer J8.7 (Pin_7)
- net LRCK: now also J8.9 (Pin_9); no longer J8.10 (Pin_10)
- net MD1/MS/AD: now also J9.8 (Pin_8); no longer J9.2 (Pin_2)
- net MD3/MC/SCL: now also J9.9 (Pin_9); no longer J9.3 (Pin_3)
- net MD4/MISO/GPIO0: now also J8.3 (Pin_3); no longer J8.4 (Pin_4)
- net MD5/GPIO1/INTA/DMIN: now also J8.4 (Pin_4); no longer J8.5 (Pin_5)
- net MD6/GPIO2/INTB/DMCLK: now also J8.5 (Pin_5); no longer J8.6 (Pin_6)
- net MDO: now also J9.7 (Pin_7); no longer J9.1 (Pin_1)
- net OSC: now also J10.1 (Pin_1); no longer J8.1 (Pin_1)
- net SCKI(3.3V): now also J8.10 (Pin_10); no longer J8.3 (Pin_3)
- net VCC: now also J10.4 (Pin_4); no longer J10.1 (Pin_1)
- net VREF: now also J9.2 (Pin_2); no longer J10.10 (Pin_10)
- net XI: now also J10.9 (Pin_9); no longer J9.9 (Pin_9)
- net XO: now also J10.10 (Pin_10); no longer J9.10 (Pin_10)
- net XO_BUFF: now also J10.6 (Pin_6); no longer J8.2 (Pin_2)
- no-connect marks 6 -> 5
Other:
- note added: "Input and output clocks"
- moved on the sheet: C16, C7, H1, H3, J10, J8

Commit message: updated potato os
Parts:
- removed J2, J3, J5, J6, J7: Conn_01x02_Male, Connector_PinHeader_2.54mm:PinHeader_1x02_P2.54mm_Vertical, symbol Connector:Conn_01x02_Male
- added J?: Conn_02x06_Row_Letter_First, symbol Connector_Generic:Conn_02x06_Row_Letter_First
Connections:
- net +1V8: now also C14.1, C16.1, C7.1, D1.2 (A), U1.11 (LDO), J?.a4 (Pin_a4)
- net VREF: now also U1.6 (VREF), J?.a3 (Pin_a3); no longer C11.2
- net XI: now also U1.10 (XI), J?.a2 (Pin_a2); no longer C3.2
- net XO: now also U1.9 (XO), J?.a1 (Pin_a1); no longer C2.1
- new net VREF_gnd: C11.2, J?.b3 (Pin_b3)
- new net XI_gnd: C3.2, J?.b2 (Pin_b2)
- new net XO_gnd: C2.1, J?.b1 (Pin_b1)

Commit message: temp
Parts:
- removed J1: Conn_01x02_Male, Connector_PinHeader_2.54mm:PinHeader_1x02_P2.54mm_Vertical, symbol Connector:Conn_01x02_Male
- removed J?: Conn_02x06_Row_Letter_First, symbol Connector_Generic:Conn_02x06_Row_Letter_First
- added J1: Conn_02x05_Row_Letter_First, Connector_PinHeader_2.54mm:PinHeader_2x05_P2.54mm_Vertical, symbol Connector_Generic:Conn_02x05_Row_Letter_First
- added R9: 4.99k, Resistor_SMD:R_0603_1608Metric_Pad0.98x0.95mm_HandSolder, symbol Device:R
Connections:
- net +3V3: now also R9.1
- net GNDD: now also J1.b4 (Pin_b4), J1.b5 (Pin_b5); no longer IC1.1 (EN)
- net VREF: now also J1.a3 (Pin_a3)
- net VREF_gnd: now also J1.b3 (Pin_b3)
- net XI: now also J1.a2 (Pin_a2)
- net XI_gnd: now also J1.b2 (Pin_b2)
- net XO: now also J1.a1 (Pin_a1)
- net XO_gnd: now also J1.b1 (Pin_b1)
- net XO_EN: now reaches IC4.5 (OE), R23.2
- net XO_EN: now also J1.a4 (Pin_a4)
- new net XI_EN: IC1.1 (EN), J1.a5 (Pin_a5), R9.2
Other:
- note added: "Ground Jumps"
- note added: "Ground jumps"
- moved on the sheet: IC1

Commit message: adc v6
Parts:
- removed C11: 1uF, Capacitor_SMD:C_0603_1608Metric_Pad1.08x0.95mm_HandSolder, symbol Device:C
- removed C2, C3: 20pF, Capacitor_SMD:C_0603_1608Metric_Pad1.08x0.95mm_HandSolder, symbol Device:C
- removed J1: Conn_02x05_Row_Letter_First, Connector_PinHeader_2.54mm:PinHeader_2x05_P2.54mm_Vertical, symbol Connector_Generic:Conn_02x05_Row_Letter_First
- removed J10, J8, J9: Conn_01x10_Male, Connector_PinHeader_2.54mm:PinHeader_1x10_P2.54mm_Vertical, symbol Connector:Conn_01x10_Male
- added C34, C35: 20pF, Capacitor_SMD:C_0603_1608Metric_Pad1.08x0.95mm_HandSolder, symbol Device:C
- added C36: 1uF, Capacitor_SMD:C_0603_1608Metric_Pad1.08x0.95mm_HandSolder, symbol Device:C
- added J1, J11, J3, J5: Conn_01x04_Pin, Connector_PinHeader_2.54mm:PinHeader_1x04_P2.54mm_Vertical, symbol Connector:Conn_01x04_Pin
- added J2: Conn_01x03_Pin, Connector_PinHeader_2.54mm:PinHeader_1x03_P2.54mm_Vertical, symbol Connector:Conn_01x03_Pin
- added J6: Conn_01x10_Pin, Connector_PinHeader_2.54mm:PinHeader_1x10_P2.54mm_Vertical, symbol Connector:Conn_01x10_Pin
- added J7: Conn_01x05_Pin, Connector_PinHeader_2.54mm:PinHeader_1x05_P2.54mm_Vertical, symbol Connector:Conn_01x05_Pin
- added J8: Conn_02x05_Top_Bottom, Connector_PinHeader_2.54mm:PinHeader_2x05_P2.54mm_Vertical, symbol Connector_Generic:Conn_02x05_Top_Bottom
Connections:
- net +1V8: now also J6.10 (Pin_10)
- net +3.3VA: now also J6.4 (Pin_4)
- net +3V3: now also J6.6 (Pin_6)
- net BCK: now also J2.3 (Pin_3)
- net DOUT: now also J2.1 (Pin_1)
- net DOUT2/MD2/MOSI/SDA: now also J3.4 (Pin_4)
- net GNDA: now also H1.1, H4.1, C36.2, J6.1 (Pin_1); no longer H2.1, H3.1
- net GNDD: now also H2.1, H3.1, C34.1, C35.1, J6.3 (Pin_3), J6.5 (Pin_5), J6.7 (Pin_7), J6.9 (Pin_9), J8.6 (Pin_6), J8.8 (Pin_8); no longer H1.1, H4.1
- net IN1: now also J5.1 (Pin_1)
- net IN2: now also J5.2 (Pin_2)
- net IN3: now also J5.3 (Pin_3)
- net IN4: now also J5.4 (Pin_4)
- net INT/GPIO3/INTC: now also J11.4 (Pin_4)
- net LRCK: now also J2.2 (Pin_2)
- net MD1/MS/AD: now also J3.2 (Pin_2)
- net MD3/MC/SCL: now also J3.3 (Pin_3)
- net MD4/MISO/GPIO0: now also J11.1 (Pin_1)
- net MD5/GPIO1/INTA/DMIN: now also J11.2 (Pin_2)
- net MD6/GPIO2/INTB/DMCLK: now also J11.3 (Pin_3)
- net MDO: now also J3.1 (Pin_1)
- net OSC: now also J7.3 (Pin_3)
- net SCKI(3.3V): now also J7.5 (Pin_5)
- net VCC: now also J6.8 (Pin_8)
- net VIN1P: now also J1.1 (Pin_1)
- net VIN2P: now also J1.2 (Pin_2)
- net VIN3P: now also J1.3 (Pin_3)
- net VIN4P: now also J1.4 (Pin_4)
- net VREF: now also J6.2 (Pin_2), J8.3 (Pin_3)
- net VREF_gnd: now also C36.1, J8.4 (Pin_4)
- net XI: now also J7.4 (Pin_4), J8.9 (Pin_9)
- net XI_gnd: now also C35.2, J8.10 (Pin_10)
- net XO: now also J7.1 (Pin_1), J8.1 (Pin_1)
- net XO_BUFF: now also J7.2 (Pin_2)
- net XO_gnd: now also C34.2, J8.2 (Pin_2)
- net XI_EN renamed XI_DIS
- net XI_DIS: now also J8.7 (Pin_7)
- net XO_EN renamed XO_DIS
- net XO_DIS: now also J8.5 (Pin_5)
Other:
- note added: "3.3V Analog LDO"
- note added: "Clocks"
- note added: "GPIO Pins"
- note added: "I2C Pins"
- note added: "I2S Pins"
- note added: "Input Pins"
- note added: "Optional XI jump to ground"
- note added: "Optional XI jump to ground to disable buffer"
- note added: "Optional XO jump to ground to disable buffer"
- note added: "Test Points"
- note added: "Test points"
- note removed: "Digital Input and Output Pins"
- note removed: "Do I want to change to digital ground because the power supply is noisy?"
- note removed: "I2C and Analog Input Pins"
- note removed: "Optional jump to ground"
- note removed: "Optional jump to ground to disable buffer"
- moved on the sheet: H1, H2, H3, H4

Commit message: mch streamer files
Parts:
- added J10, J12, J13, J9: Eurorack_Mono_Jack, winterbloom:AudioJack_WQP518MA, symbol winterbloom:Eurorack_Mono_Jack
Connections:
- net GNDA: now also J10.S (Sleeve), J12.S (Sleeve), J13.S (Sleeve), J9.S (Sleeve)
- net IN1: now also J9.T (Tip)
- net IN2: now also J10.T (Tip)
- net IN3: now also J12.T (Tip)
- net IN4: now also J13.T (Tip)
- no-connect marks 5 -> 9
Other:
- note added: "TN: NC T: Tip (signal) S: GND"
- note added: "TN: a switch connected to the input. Could be used to change between jack inputs and CV inputs. NC for now."

Commit message: jack
Parts:
- removed C17: .01uF, Capacitor_SMD:C_0603_1608Metric_Pad1.08x0.95mm_HandSolder, symbol Device:C
- removed C28, C29: 0.1uF, Capacitor_SMD:C_0603_1608Metric_Pad1.08x0.95mm_HandSolder, symbol Device:C
- removed C34, C35: 20pF, Capacitor_SMD:C_0603_1608Metric_Pad1.08x0.95mm_HandSolder, symbol Device:C
- removed C36: 1uF, Capacitor_SMD:C_0603_1608Metric_Pad1.08x0.95mm_HandSolder, symbol Device:C
- removed IC1: SN74AUC1G126DCKR, custom_lib:SOT65P210X110-5N, symbol custom_lib:SN74AUC1G126DCKR
- removed IC4: TXB0101DBVT, custom_lib:SOT95P280X145-6N, symbol custom_lib:TXB0101DBVT
- removed J10, J12, J13, J9: Eurorack_Mono_Jack, winterbloom:AudioJack_WQP518MA, symbol winterbloom:Eurorack_Mono_Jack
- removed J11: Conn_01x04_Pin, Connector_PinHeader_2.54mm:PinHeader_1x04_P2.54mm_Vertical, symbol Connector:Conn_01x04_Pin
- removed J2: Conn_01x03_Pin, Connector_PinHeader_2.54mm:PinHeader_1x03_P2.54mm_Vertical, symbol Connector:Conn_01x03_Pin
- removed J4: USB_B_Micro, Connector_USB:USB_Micro-B_Wuerth_629105150521, symbol Connector:USB_B_Micro
- removed J7: Conn_01x05_Pin, Connector_PinHeader_2.54mm:PinHeader_1x05_P2.54mm_Vertical, symbol Connector:Conn_01x05_Pin
- removed J8: Conn_02x05_Top_Bottom, Connector_PinHeader_2.54mm:PinHeader_2x05_P2.54mm_Vertical, symbol Connector_Generic:Conn_02x05_Top_Bottom
- removed R23: 4.99k, Resistor_SMD:R_0603_1608Metric_Pad0.98x0.95mm_HandSolder, symbol Device:R
- removed Y2: ASE-22.000MHZ-ET, custom_lib:ASE24000MHZET, symbol custom_lib:ASE-22.000MHZ-ET
- added J2: Conn_01x04_Pin, symbol Connector:Conn_01x04_Pin
- added R10: 100k, Resistor_SMD:R_0603_1608Metric_Pad0.98x0.95mm_HandSolder, symbol Device:R
- R5, R6: value 100 -> 100k
- R7, R8: value 100 -> 800
- R9: value 4.99k -> 100k
Connections:
- net INT/GPIO3/INTC is gone; now on net GNDD: U1.19 (GPIO3/INTC)
- net MD4/MISO/GPIO0 is gone; now on net GNDD: U1.22 (MISO/GPIO0/DMIN2)
- net MD5/GPIO1/INTA/DMIN is gone; now on net GNDD: U1.21 (GPIO1/INTA/DMIN)
- net MD6/GPIO2/INTB/DMCLK is gone; now on net GNDD: U1.20 (GPIO2/INTB/DMCLK)
- net XI is gone; now on net GNDD: U1.10 (XI)
- net XI_DIS is gone; now on net VREF: R9.2
- net XO is gone; now on net GNDD: U1.9 (XO)
- net +3.3VA: now also R10.2
- net +3V3: no longer R9.1
- net BCK: now also J2.3 (Pin_3)
- net DOUT: now also J2.1 (Pin_1)
- net GNDA: now also R9.1
- net LRCK: now also J2.2 (Pin_2)
- net SCKI(3.3V): now also J2.4 (Pin_4)
- net VREF: now also R10.1
- no-connect marks 9 -> 2
Other:
- note added: "need to determine. tie down with resistors"
- note added: "tie down with resistors"
- note removed: "22MHz Crystal Oscillator"
- note removed: "Clocks"
- note removed: "D+ and D- can be used for serial communication, but we are not"
- note removed: "GPIO Pins"
- note removed: "Ground Jumps"
- note removed: "Ground jumps"
- note removed: "Input and output clocks"
- note removed: "Optional XI jump to ground"
- note removed: "Optional XI jump to ground to disable buffer"
- note removed: "Optional XO jump to ground to disable buffer"
- note removed: "Output = .9 *VDDhigh"
- note removed: "Output enable (OE): High - on Low - off"
- note removed: "Steps 3.3V oscillator down to 1.8V logic"
- note removed: "TN: NC T: Tip (signal) S: GND"
- note removed: "TN: a switch connected to the input. Could be used to change between jack inputs and CV inputs. NC for now."
- note removed: "Test point or jump to ground"
- note removed: "XI Buffer"
- note removed: "XO Buffer"
- moved on the sheet: C1, C24, C25, C4, C5, C6, C9, D2, D3, D4, FB1, H1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
