File: Transmitter/Transmitter.kicad_sch (KiCad schematic)
At the start: 18 parts, among them IC1 TORX1950A_F_, IC2 TORX1950A_F_, IC3 TORX1950A_F_, J1 Conn_01x08_Male

Commit message: Version 3 transmitter
Parts:
- added H1, H2: MountingHole_Pad, MountingHole:MountingHole_3.2mm_M3_ISO7380_Pad, symbol Mechanical:MountingHole_Pad
- added Q1, Q2, Q3, Q4, Q5: BSS138, Package_TO_SOT_SMD:SOT-23, symbol Transistor_FET:BSS138
- IC1, IC2, IC3: footprint KiCad:TORX1950AF -> TOTX and TORX:TORX1950AF
- LED1, LED2: footprint KiCad:TOTX1950AF -> TOTX and TORX:TOTX1950AF
- R3: value 1.5k -> 10k
Connections:
- net GND: now also J1.1 (Pin_1), H1.1, H2.1; no longer J1.2 (Pin_2)
- net VCC: now also J1.2 (Pin_2), Q4.2 (S), Q5.2 (S); no longer J1.1 (Pin_1)
- net +3.3V: now reaches J1.3 (Pin_3)
- net +3.3V: now also Q1.2 (S), Q2.2 (S), Q3.2 (S)
- net IN1: no longer names the net of LED1.4 (INPUT)
- net IN1: now also Q4.3 (D); no longer J1.7 (Pin_7)
- net IN2: no longer names the net of LED2.4 (INPUT)
- net IN2: now also Q5.3 (D); no longer J1.8 (Pin_8)
- net OUT1: no longer names the net of IC1.1 (OUTPUT)
- net OUT1: now also Q1.1 (G); no longer J1.4 (Pin_4)
- net OUT2: no longer names the net of IC2.1 (OUTPUT)
- net OUT2: now also Q2.1 (G); no longer J1.5 (Pin_5)
- net OUT3: no longer names the net of IC3.1 (OUTPUT)
- net OUT3: now also Q3.1 (G); no longer J1.6 (Pin_6)
- new net IN 1: J1.4 (Pin_4), Q4.1 (G)
- new net IN 2: J1.5 (Pin_5), Q5.1 (G)
- new net OUT 1: J1.8 (Pin_8), Q1.3 (D)
- new net OUT 2: J1.7 (Pin_7), Q2.3 (D)
- new net OUT 3: J1.6 (Pin_6), Q3.3 (D)
- no-connect marks 11 -> 10
Other:
- moved on the sheet: C1, C2, C5, D1, IC1, IC2, L1, L2, LED2, R2, R3
